Commit message: Update from boss

File: robot_description/urdf/robot.urdf (robot description, URDF)
Before this commit: robot Robot_Arm, 3 links, 2 joints
Links:
- link base_link: geometry visual mesh filename=package://robot_description/STL/base.stl scale=0.001 0.001 0.001
- link link1: geometry visual mesh filename=package://robot_description/STL/slider.stl scale=0.001 0.001 0.001
- link link2: geometry visual mesh filename=package://robot_description/STL/link2.stl scale=0.001 0.001 0.001
Joints:
- joint joint1: axis 0 1 0 -> 0 0 1; origin xyz=0 0 0.075 rpy=1.56 0 0 -> xyz=0 0 0 rpy=0 0 0
- joint joint2: origin xyz=0 0 0.075 rpy=1.56 0 0 -> xyz=0 0 0 rpy=0 0 0
